File: eternal_nrf_pcb/eternal_nrf_pcb.kicad_pcb (KiCad board)
At the start: 2 copper layers, 27.5 x 42.5 mm, 49 parts, among them J1 Conn_01x05_Pin, Q1 IRLML6244, Q2 IRLML6402, SW1 SW_Push, U1 BQ25504, U2 nRF52810-QCxx, U3 DRV5032DU, U4 SHTC3, Y1 Crystal_GND24

Commit message: almost final layout
Parts:
- added C18: 100uF, Capacitor_SMD:C_1210_3225Metric, F.Cu at (128.1, 85.3)
- added C19: 100uF, Capacitor_SMD:C_1210_3225Metric, F.Cu at (128.1, 89.1)
- added L5: 6.8uH, Inductor_SMD:L_0402_1005Metric_Pad0.77x0.64mm_HandSolder, F.Cu at (145.8, 115.6)
- AE1: value Antenna_Dipole -> RFANT3216120A5T
- BT1: value Battery_Cell -> Battery
- J1: footprint Connector_PinHeader_2.00mm:PinHeader_1x05_P2.00mm_Vertical -> Connector_PinHeader_2.54mm:PinHeader_1x05_P2.54mm_Vertical
- R13: value 6.8K -> 4.7K
- R4: value 5.76M -> 6.34M
- TP1: value SLR+ -> S+
- TP2: value SLR- -> S-
- moved TP2 22.6 mm to (150.5, 107.1)
- moved D1 19.9 mm to (138.8, 116.5), turned to 180 degrees
- moved R13 15.4 mm to (134.4, 111.2), turned to 180 degrees
- moved SW1 9.20 mm to (127.3, 96.0)
- moved JP1 8.59 mm to (138.9, 99.7)
- moved R7 8.58 mm to (144.1, 88.3), turned to 180 degrees
- moved R5 5.93 mm to (142.7, 95.0), turned to 90 degrees
- moved L4 3.81 mm to (139.1, 104.9), turned to -90 degrees
- moved TP1 2.70 mm to (150.5, 85.4)
- moved C13 2.59 mm to (143.9, 103.2)
- moved J1 2.59 mm to (127.6, 104.8)
- moved C12 2.42 mm to (143.9, 108.8), turned to 180 degrees
- moved L3 2.30 mm to (137.7, 104.4), turned to 90 degrees
- moved C14 2.24 mm to (140.2, 104.9)
- moved R6 2.20 mm to (141.1, 95.0)
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Connections:
- L2 pad 1: Net-(AE1-Pad1) -> Net-(L2-Pad1)

Commit message: almost final layout
Parts:
- turned L5 to 180 degrees
Changed lines of the file:
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@@
 	(footprint "Inductor_SMD:L_0402_1005Metric_Pad0.77x0.64mm_HandSolder"
 		(layer "F.Cu")
-		(at 145.8275 115.6)
+		(at 145.8275 115.6 180)
 		(descr "Inductor SMD 0402 (1005 Metric), square (rectangular) end terminal, IPC-7351 nominal with elongated pad for handsoldering. (Body size source: http://www.tortai-tech.com/upload/download/2011102023233369053.pdf)")
 		(tags "inductor handsolder")
@@
 		(duplicate_pad_numbers_are_jumpers no)
 		(fp_line
-			(start -0.1002 -0.36)
-			(end 0.1002 -0.36)
+			(start -0.1002 0.36)
+			(end 0.1002 0.36)
 			(stroke
 				(width 0.12)
@@
 		)
 		(fp_line
-			(start -0.1002 0.36)
-			(end 0.1002 0.36)
+			(start -0.1002 -0.36)
+			(end 0.1002 -0.36)
 			(stroke
 				(width 0.12)
@@
 		)
 		(pad "1" smd roundrect
-			(at -0.5725 0)
+			(at -0.5725 0 180)
 			(size 0.765 0.64)
 			(layers "F.Cu" "F.Mask" "F.Paste")
@@
 		)
 		(pad "2" smd roundrect
-			(at 0.5725 0)
+			(at 0.5725 0 180)
 			(size 0.765 0.64)
 			(layers "F.Cu" "F.Mask" "F.Paste")

Commit message: somewhat complete wiring
Parts:
- moved R10 4.64 mm to (146.9, 97.8), turned to -90 degrees
- moved C4 3.96 mm to (146.9, 101.1)
- moved C3 1.25 mm to (138.6, 86.5), turned to 90 degrees
- moved C7 0.97 mm to (143.3, 112.8)
- moved L2 0.97 mm to (144.5, 112.8)
- moved C9 0.33 mm to (135.6, 114.1)
- moved C8 0.33 mm to (137.0, 113.8)
- moved U4 0.24 mm to (150.4, 77.1), turned to 0 degrees
- moved C18 0.23 mm to (127.9, 85.3), turned to 180 degrees
- moved C19 0.23 mm to (127.9, 89.1), turned to 180 degrees
- moved C11 0.20 mm to (143.9, 109.8)
- moved R11 0.20 mm to (138.9, 114.4)
- moved R12 0.20 mm to (140.1, 114.4)
- moved L5 0.12 mm to (145.9, 115.7)
- turned C1 to 180 degrees
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Routing:
- net Net-(BT1-+): track 0.00 -> 60.0 mm, vias 0 -> 4
- net MAG: track 0.00 -> 57.2 mm, vias 0 -> 2
- net SHT_VCC: track 0.00 -> 52.8 mm, vias 0 -> 3
- net SCL: track 0.00 -> 51.9 mm, vias 0 -> 2
- net SDA: track 0.00 -> 51.9 mm, vias 0 -> 2
- net RST: track 0.00 -> 35.1 mm, vias 0 -> 2
- net VCC: track 0.00 -> 34.3 mm, vias 0 -> 6
- net BUTTON: track 0.00 -> 33.4 mm, vias 0 -> 2
- net Net-(U1-VIN_DC): track 0.00 -> 31.4 mm
- net Net-(Q2-S): track 0.00 -> 27.6 mm, vias 0 -> 2
- net GND: track 0.00 -> 25.1 mm, vias 0 -> 22
- net DIO: track 0.00 -> 17.0 mm, vias 0 -> 1
- net Net-(U1-VRDIV): track 0.00 -> 16.1 mm
- net CLK: track 0.00 -> 15.5 mm, vias 0 -> 1
- net Net-(Q1-G): track 0.00 -> 15.3 mm
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- added copper zone on B.Cu, net GND
- added copper zone on F.Cu, net GND
- added copper zone on In1.Cu, net GND
- added copper zone on F.Cu, net VCC
- added copper zone on In2.Cu, net VCC
Other:
- copper layers 2 -> 4

Commit message: almost complete design, touch ups are pending
Parts:
- moved C7 2.06 mm to (144.1, 110.8), turned to 0 degrees
- moved L2 0.41 mm to (144.5, 113.2)
Routing:
- net GND: track 25.1 -> 55.1 mm, vias 22 -> 20
- net Net-(BT1-+): track 60.0 -> 43.9 mm, vias 4 -> 0
- net Net-(JP1-B): track 12.9 -> 17.9 mm
- net RST: track 35.1 -> 31.6 mm
- net SDA: track 51.9 -> 50.9 mm
- net Net-(U2-ANT): track 3.88 -> 4.40 mm
- net Net-(U1-VIN_DC): track 31.4 -> 31.5 mm, vias 0 -> 2

Commit message: change fonts
Parts:
- moved C7 0.15 mm to (143.9, 110.8)
Routing:
- net GND: track 55.1 -> 57.4 mm
Other:
- board text added: "CLK"
- board text added: "DIO"
- board text added: "GND"
- board text added: "RST"
- board text added: "VCC"

Commit message: final pcb (rev 1 :))
Routing:
- net GND: track 57.4 -> 60.2 mm, vias 20 -> 43
Other:
- board text added: "Eternal nRF"
- board text added: "MT"
- board text added: "Rev. 1, 9th May 2026 Madhukar Temba"

Commit message: complete board
Parts:
- added C20: 22pF, Capacitor_SMD:C_0402_1005Metric_Pad0.74x0.62mm_HandSolder, F.Cu at (131.5, 107.4)
- added C21: 22pF, Capacitor_SMD:C_0402_1005Metric_Pad0.74x0.62mm_HandSolder, F.Cu at (133.4, 104.7)
- added Y2: Crystal, Crystal:Crystal_SMD_3215-2Pin_3.2x1.5mm, F.Cu at (133.4, 107.4)
- J1: value Conn_01x05_Pin -> Conn_01x07_Pin; footprint Connector_PinHeader_2.54mm:PinHeader_1x05_P2.54mm_Vertical -> Connector_PinHeader_2.54mm:PinHeader_1x07_P2.54mm_Vertical
- moved J1 4.61 mm to (127.1, 100.3)
- moved C10 1.90 mm to (135.4, 106.2), turned to -90 degrees
- moved SW1 0.68 mm to (127.3, 95.3)
Connections:
- J1 pad 2: RST -> TX
- J1 pad 3: DIO -> RX
- J1 pad 4: CLK -> RST
- J1 pad 5: VCC -> DIO
- U2 pad 2: unconnected-(U2-P0.00/XL1-Pad2) -> Net-(U2-P0.00/XL1)
- U2 pad 3: unconnected-(U2-P0.01/XL2-Pad3) -> Net-(U2-P0.01/XL2)
- U2 pad 4: unconnected-(U2-P0.04/AIN2-Pad4) -> TX
- U2 pad 5: unconnected-(U2-P0.05/AIN3-Pad5) -> RX
Routing:
- net TX: track 0.00 -> 14.5 mm, vias 0 -> 1
- net RX: track 0.00 -> 13.6 mm, vias 0 -> 1
- net Net-(U2-P0.00/XL1): track 0.00 -> 6.37 mm
- net Net-(U2-P0.01/XL2): track 0.00 -> 5.44 mm
- net CLK: track 15.5 -> 17.1 mm
- net VCC: track 34.3 -> 35.7 mm
- net RST: track 31.6 -> 30.5 mm
- net BUTTON: track 33.4 -> 34.0 mm
- net GND: vias 43 -> 39
Other:
- board text added: "RX"
- board text added: "TX"
